File: kicad/kichenclock.sch (KiCad schematic (older format))
At the start: 20 parts, among them CON1 AVR-ISP-6, J1 pwr_1v5, J2 OLED_DISPLAY, SW1 DOWN, SW2 OK, SW3 UP, U1 LT1073, U2 ATTINY85-20SU

Commit message: kicad files done
Parts:
- removed D1: 1N5818, Diode_THT:D_DO-41_SOD81_P10.16mm_Horizontal, symbol Diode:1N5818
- removed J?: PROG, symbol Connector_Generic:Conn_01x02
- removed R2, R3, R6: 1K, symbol Device:R
- added D1: SB120, Diode_SMD:D_SMA_Handsoldering, symbol Diode:SB120
- added L2: 1uH, Inductor_SMD:L_0805_2012Metric_Pad1.15x1.50mm_HandSolder, symbol Device:L
- added MK1, MK2: Mounting_Hole_PAD, MountingHole:MountingHole_3mm_Pad, symbol Mechanical:Mounting_Hole_PAD
- C1: footprint (none) -> Capacitor_Tantalum_SMD:CP_EIA-6032-20_AVX-F_Pad2.24x2.40mm_HandSolder
- C2: footprint (none) -> Capacitor_Tantalum_SMD:CP_EIA-6032-20_AVX-F
- C3: footprint (none) -> Capacitor_SMD:C_0805_2012Metric_Pad1.15x1.50mm_HandSolder
- CON1: footprint (none) -> Connector_PinSocket_2.54mm:PinSocket_2x03_P2.54mm_Vertical
- J1: footprint (none) -> Connector_PinHeader_2.54mm:PinHeader_1x02_P2.54mm_Vertical
- J2: footprint (none) -> modules_copy:oled_128x32
- L1: footprint (none) -> Choke_SMD:Choke_CD75
- R1, R4, R5: footprint (none) -> Resistor_SMD:R_1206_3216Metric
- SW1, SW2, SW3: footprint (none) -> Button_Switch_THT:SW_PUSH_6mm
- U1: footprint MODULE -> Package_SO:SOIC-8_3.9x4.9mm_P1.27mm
- U2: footprint Housings_SOIC:SOIC-8_3.9x4.9mm_Pitch1.27mm -> Package_SO:SOIC-8_3.9x4.9mm_P1.27mm
Connections:
- net +3V3: now also J2.3 (Pin_3), D1.1 (K); no longer J2.2 (Pin_2)
- net GND: now also J2.4 (Pin_4), MK1.1, MK2.1; no longer J2.1 (Pin_1)
- net MISO: now also SW1.1
- net MOSI: now also J2.1 (Pin_1); no longer J2.4 (Pin_4)
- net SCK: now also J2.2 (Pin_2); no longer J2.3 (Pin_3)
- net at L1.1, R1.1, U1.2 (Vin): now also L2.2; no longer J1.2 (Pin_2)
- net at L1.2, U1.3 (SW1): now also D1.2 (A)
- new net: J1.2 (Pin_2), L2.1
Other:
- moved on the sheet: C1, J1, J2, L1, R1, R4, R5, SW1, SW2, SW3, U1
